File: 1.kicad_pcb (KiCad board)
At the start: 2 copper layers, 64 parts, among them J1 ValveOUT, J10 PD6, J2 MotorOUT, J3 PumpOUT, J4 220V_IN, J5 ISCP, J6 LedOUT, J7 FloatOUT, J8 SwitchOUT, J9 ButtonOUT, Q1 BT136, Q2 BT136, Q3 BT136, SW1 SW_Push, U1 ATmega8A-AU, U2 MOC3023M, U3 MOC3023M, U4 MOC3023M, Y1 16MHz

Commit message: Add files via upload
Parts:
- R1, R2: footprint Resistors_SMD:R_1206 -> Resistors_SMD:R_0805
- moved C3 29.2 mm to (37.2, 78.0), turned to 0 degrees
- moved R1 9.52 mm to (49.3, 68.2), turned to 270 degrees
- moved + 9.08 mm to (62.3, 103.2), turned to 180 degrees
- moved R4 8.46 mm to (31.9, 102.4), turned to 0 degrees
- moved R5 8.46 mm to (51.9, 102.4), turned to 0 degrees
- moved R3 8.45 mm to (42.0, 102.4), turned to 0 degrees
- moved R6 3.23 mm to (62.3, 57.9), turned to 0 degrees
- moved R7 0.82 mm to (77.1, 46.8)
- renumbered R22 to +, R23 to -, REF** to AC-DC_5V
Routing:
- net Earth: track 315.9 -> 137.5 mm, vias 2 -> 1
- net +5V: track 132.7 -> 151.5 mm, vias 10 -> 0
- net /RST: track 32.2 -> 24.1 mm, vias 2 -> 0
- net /Switch: track 24.9 -> 28.7 mm
- net /ValvePin: track 59.4 -> 56.5 mm, vias 2 -> 0
- net Net-(D1-Pad2): track 3.95 -> 2.14 mm
- net Net-(J10-Pad1): track 7.28 -> 5.67 mm
- net /Float: track 24.9 -> 26.4 mm
- net /PD6: track 27.9 -> 26.4 mm
- net Net-(R7-Pad1): track 3.80 -> 4.67 mm
- net /MOSI: track 28.2 -> 27.4 mm, vias 0 -> 1
- net /Button: track 30.1 -> 30.8 mm
- added copper zone on F.Cu, net Earth
Other:
- board text added: "+5V"
- board text added: "GND"
- board text added: "MISO"
- board text added: "MOSI"
- board text added: "RST"
- board text added: "SCK"

Commit message: Add files via upload
Parts:
- F1: footprint Library:MyBladeFuse -> Fuse_Holders_and_Fuses:Fuse_TE5_Littlefuse-395Series
- moved F1 3.59 mm to (27.9, 53.1)
Routing:
- net /220_In2: track 197.2 -> 212.8 mm
- net /220_In1: track 184.8 -> 183.8 mm
- net Net-(F1-Pad1): track 10.4 -> 9.81 mm
Changed lines of the file:
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@@
   (general
     (thickness 1.6)
-    (drawings 10)
-    (tracks 348)
+    (drawings 12)
+    (tracks 353)
     (zones 0)
     (modules 64)
@@
     (43 Eco2.User user hide)
     (44 Edge.Cuts user)
-    (45 Margin user hide)
+    (45 Margin user)
     (46 B.CrtYd user hide)
     (47 F.CrtYd user hide)
@@
   )
   (setup
-    (last_trace_width 1)
+    (last_trace_width 1.5)
     (user_trace_width 0.5)
     (user_trace_width 0.6)
@@
     (visible_elements 7FFFFF7F)
     (pcbplotparams
-      (layerselection 0x010f0_ffffffff)
+      (layerselection 0x030f0_ffffffff)
       (usegerberextensions false)
       (usegerberattributes false)
@@
     (add_net "Net-(U4-Pad5)")
   )
+  (module Fuse_Holders_and_Fuses:Fuse_TE5_Littlefuse-395Series (layer F.Cu)
+    (at 27.95 53.15 90)
+    (descr "Fuse, TE5, Littlefuse/Wickmann, No. 460, No560,")
+    (tags "Fuse TE5 Littlefuse/Wickmann No. 460 No560 ")
+    (fp_text reference F1 (at 1.86 0.02 180) (layer F.SilkS)
+      (effects (font (size 1 1) (thickness 0.15)))
+    )
+    (fp_text value Fuse (at 4 3.05 90) (layer F.Fab)
+      (effects (font (size 1 1) (thickness 0.15)))
+    )
+    (fp_line (start -1.71 2) (end 6.79 2) (layer F.Fab) (width 0.1))
+    (fp_line (start 6.79 2) (end 6.79 -2) (layer F.Fab) (width 0.1))
+    (fp_line (start 6.79 -2) (end -1.71 -2) (layer F.Fab) (width 0.1))
+    (fp_line (start -1.71 -2) (end -1.71 2) (layer F.Fab) (width 0.1))
+    (fp_line (start -1.96 -2.25) (end 7.04 -2.25) (layer F.CrtYd) (width 0.05))
+    (fp_line (start -1.96 -2.25) (end -1.96 2.25) (layer F.CrtYd) (width 0.05))
+    (fp_line (start 7.04 2.25) (end 7.04 -2.25) (layer F.CrtYd) (width 0.05))
+    (fp_line (start 7.04 2.25) (end -1.96 2.25) (layer F.CrtYd) (width 0.05))
+    (fp_line (start -1.83 -2.12) (end 6.91 -2.12) (layer F.SilkS) (width 0.12))
+    (fp_line (start -1.83 -2.12) (end -1.83 2.12) (layer F.SilkS) (width 0.12))
+    (fp_line (start 6.91 2.12) (end 6.91 -2.12) (layer F.SilkS) (width 0.12))
+    (fp_line (start 6.91 2.12) (end -1.83 2.12) (layer F.SilkS) (width 0.12))
+    (pad 1 thru_hole circle (at 0 0 90) (size 2 2) (drill 1) (layers *.Cu *.Mask)
+      (net 15 "Net-(F1-Pad1)"))
+    (pad 2 thru_hole circle (at 5.08 0.01 90) (size 2 2) (drill 1) (layers *.Cu *.Mask)
+      (net 40 /220_In1))
+  )
   (module Housings_QFP:LQFP-32_7x7mm_Pitch0.8mm (layer B.Cu)
     (at 49.3 76.31 180)
@@
     (pad 1 thru_hole circle (at 0 0 90) (size 2 2) (drill 1.1) (layers *.Cu *.Mask))
   )
-  (module Library:MyBladeFuse (layer F.Cu)
-    (at 27.86 56.74 90)
-    (descr "car blade fuse mini")
-    (tags "car blade fuse mini")
-    (fp_text reference F1 (at 1.86 0.02 180) (layer F.SilkS)
-      (effects (font (size 1 1) (thickness 0.15)))
-    )
-    (fp_text value Fuse (at 4 3.05 90) (layer F.Fab)
-      (effects (font (size 1 1) (thickness 0.15)))
-    )
-    (fp_line (start 10.9 2.2) (end -3 2.2) (layer F.CrtYd) (width 0.05))
-    (fp_line (start 10.9 2.2) (end 10.9 -2.2) (layer F.CrtYd) (width 0.05))
-    (fp_line (start -3 -2.2) (end -3 2.2) (layer F.CrtYd) (width 0.05))
-    (fp_line (start -3 -2.2) (end 10.9 -2.2) (layer F.CrtYd) (width 0.05))
-    (fp_line (start 2.4 -2) (end 5.6 -2) (layer F.SilkS) (width 0.12))
-    (fp_line (start 5.6 2) (end 2.4 2) (layer F.SilkS) (width 0.12))
-    (fp_line (start 3.25 0) (end 4.85 0) (layer F.SilkS) (width 0.12))
-    (fp_line (start -1.55 1.95) (end -1.55 -1.95) (layer F.Fab) (width 0.1))
-    (fp_line (start 9.55 1.95) (end -1.55 1.95) (layer F.Fab) (width 0.1))
-    (fp_line (start 9.55 -1.95) (end 9.55 1.95) (layer F.Fab) (width 0.1))
-    (fp_line (start -1.55 -1.95) (end 9.55 -1.95) (layer F.Fab) (width 0.1))
-    (pad 2 thru_hole oval (at 8 0 90) (size 2 2) (drill 1) (layers *.Cu *.Mask)
-      (net 40 /220_In1))
-    (pad 1 thru_hole oval (at 0 0 90) (size 2 2) (drill 1) (layers *.Cu *.Mask)
-      (net 15 "Net-(F1-Pad1)"))
-    (model Fuse_Holders_and_Fuses.3dshapes/BladeFuse-Mini.wrl
-      (offset (xyz 4.063999938964844 0 0))
-      (scale (xyz 0.39 0.39 0.39))
-      (rotate (xyz 0 0 0))
-    )
-  )
   (module Connectors_Terminal_Blocks:TerminalBlock_Altech_AK300-2_P5.00mm (layer F.Cu)
     (at 18.66 26.48 270)
@@
     )
   )
+  (gr_line (start 12.02 105.01) (end 112.02 104.99) (layer B.SilkS) (width 0.12))
+  (gr_line (start 12.01 12) (end 112.01 11.98) (layer B.SilkS) (width 0.12))
+  (gr_line (start 12.01 12) (end 12.02 105.01) (layer B.SilkS) (width 0.12))
+  (gr_line (start 112.01 11.98) (end 112.02 104.99) (layer B.SilkS) (width 0.12))
   (gr_text MOSI (at 24.45 77.64) (layer F.SilkS)
     (effects (font (size 1 1) (thickness 0.15)))
@@
   )
   (gr_line (start 12.02 105.01) (end 12.01 12) (layer Margin) (width 0.12))
-  (gr_line (start 112.01 105.01) (end 12.02 105.01) (layer Margin) (width 0.12))
-  (gr_line (start 112.01 11.98) (end 112.01 105.01) (layer Margin) (width 0.12))
   (gr_line (start 12.01 12) (end 112.01 11.98) (layer Margin) (width 0.12))
   (segment (start 59.9 75.71) (end 59.9 79.18) (width 0.7) (layer B.Cu) (net 1))
@@
   (segment (start 52.89 102.43) (end 53.84 102.43) (width 0.6) (layer B.Cu) (net 13))
   (segment (start 63.24 57.93) (end 63.24 55.79) (width 0.7) (layer B.Cu) (net 14))
-  (segment (start 21.129 56.74) (end 18.569 54.18) (width 2) (layer B.Cu) (net 15))
-  (segment (start 27.86 56.74) (end 21.129 56.74) (width 2) (layer B.Cu) (net 15))
+  (segment (start 19.599 53.15) (end 18.569 54.18) (width 1.5) (layer B.Cu) (net 15))
+  (segment (start 27.95 53.15) (end 19.599 53.15) (width 1.5) (layer B.Cu) (net 15))
   (segment (start 30.28 75.25) (end 34.18 71.35) (width 0.8) (layer B.Cu) (net 16))
   (segment (start 44.670001 70.350001) (end 42.039999 70.350001) (width 0.7) (layer B.Cu) (net 16))
@@
   (segment (start 69.05 34.26) (end 66.45 31.66) (width 2) (layer B.Cu) (net 40))
   (segment (start 69.05 34.36) (end 66.24 37.17) (width 2) (layer B.Cu) (net 40))
-  (segment (start 31.478 48.74) (end 32.134 48.084) (width 2) (layer B.Cu) (net 40))
-  (segment (start 27.86 48.74) (end 31.478 48.74) (width 2) (layer B.Cu) (net 40))
-  (segment (start 27.86 44.18) (end 27.86 48.74) (width 2) (layer B.Cu) (net 40))
   (segment (start 38.998 34.544792) (end 38.998 33.272) (width 1.5) (layer B.Cu) (net 40))
   (segment (start 38.998 35.042) (end 38.998 34.544792) (width 1.5) (layer B.Cu) (net 40))
@@
   (segment (start 66.45 31.66) (end 52.389999 17.599999) (width 1.5) (layer B.Cu) (net 40))
   (segment (start 52.389999 17.599999) (end 45.839999 17.599999) (width 1.5) (layer B.Cu) (net 40))
-  (segment (start 32.134 53.164) (end 26.834 53.164) (width 2) (layer B.Cu) (net 41))
-  (segment (start 22.85 49.18) (end 18.569 49.18) (width 2) (layer B.Cu) (net 41))
-  (segment (start 26.834 53.164) (end 22.85 49.18) (width 2) (layer B.Cu) (net 41))
+  (segment (start 32.12 48.07) (end 32.134 48.084) (width 1.5) (layer B.Cu) (net 40))
+  (segment (start 27.96 48.07) (end 32.12 48.07) (width 1.5) (layer B.Cu) (net 40))
+  (segment (start 27.96 44.28) (end 27.86 44.18) (width 1.5) (layer B.Cu) (net 40))
+  (segment (start 27.96 48.07) (end 27.96 44.28) (width 1.5) (layer B.Cu) (net 40))
   (segment (start 18.66 31.48) (end 15.18 31.48) (width 1.5) (layer B.Cu) (net 41))
   (segment (start 15.18 31.48) (end 14.43 30.73) (width 1.5) (layer B.Cu) (net 41))
@@
   (segment (start 18.66 49.089) (end 18.569 49.18) (width 2) (layer B.Cu) (net 41))
   (segment (start 18.66 31.48) (end 18.66 49.089) (width 2) (layer B.Cu) (net 41))
+  (segment (start 17.579 49.18) (end 14.675 52.084) (width 1.5) (layer B.Cu) (net 41))
+  (segment (start 18.569 49.18) (end 17.579 49.18) (width 1.5) (layer B.Cu) (net 41))
+  (segment (start 14.675 52.084) (end 14.675 55.925) (width 1.5) (layer B.Cu) (net 41))
+  (segment (start 14.675 55.925) (end 16.975 58.225) (width 1.5) (layer B.Cu) (net 41))
+  (segment (start 16.975 58.225) (end 29.475 58.225) (width 1.5) (layer B.Cu) (net 41))
+  (segment (start 32.134 55.566) (end 32.134 53.164) (width 1.5) (layer B.Cu) (net 41))
+  (segment (start 29.475 58.225) (end 32.134 55.566) (width 1.5) (layer B.Cu) (net 41))
   (segment (start 79.03 46.77) (end 81.61 49.35) (width 0.7) (layer B.Cu) (net 42))
   (segment (start 78.01 46.77) (end 79.03 46.77) (width 0.7) (layer B.Cu) (net 42))

Commit message: Add files via upload
Other:
- board outline added: 100 x 93 mm
Changed lines of the file:
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@@
   (general
     (thickness 1.6)
-    (drawings 12)
+    (drawings 10)
     (tracks 353)
     (zones 0)
@@
   )
   (setup
-    (last_trace_width 1.5)
+    (last_trace_width 1)
     (user_trace_width 0.5)
     (user_trace_width 0.6)
@@
     (visible_elements 7FFFFF7F)
     (pcbplotparams
-      (layerselection 0x030f0_ffffffff)
+      (layerselection 0x010f0_ffffffff)
       (usegerberextensions false)
       (usegerberattributes false)
@@
     )
   )
-  (gr_line (start 12.02 105.01) (end 112.02 104.99) (layer B.SilkS) (width 0.12))
-  (gr_line (start 12.01 12) (end 112.01 11.98) (layer B.SilkS) (width 0.12))
-  (gr_line (start 12.01 12) (end 12.02 105.01) (layer B.SilkS) (width 0.12))
-  (gr_line (start 112.01 11.98) (end 112.02 104.99) (layer B.SilkS) (width 0.12))
+  (gr_line (start 12.02 105.01) (end 112.02 104.99) (layer Edge.Cuts) (width 0.12))
+  (gr_line (start 112.01 11.98) (end 112.02 104.99) (layer Edge.Cuts) (width 0.12))
   (gr_text MOSI (at 24.45 77.64) (layer F.SilkS)
     (effects (font (size 1 1) (thickness 0.15)))
@@
     (effects (font (size 1 1) (thickness 0.15)))
   )
-  (gr_line (start 12.02 105.01) (end 12.01 12) (layer Margin) (width 0.12))
-  (gr_line (start 12.01 12) (end 112.01 11.98) (layer Margin) (width 0.12))
+  (gr_line (start 12.02 105.01) (end 12.01 12) (layer Edge.Cuts) (width 0.12))
+  (gr_line (start 12.01 12) (end 112.01 11.98) (layer Edge.Cuts) (width 0.12))
   (segment (start 59.9 75.71) (end 59.9 79.18) (width 0.7) (layer B.Cu) (net 1))
   (segment (start 54.87 78.31) (end 53.55 78.31) (width 0.6) (layer B.Cu) (net 1))

Commit message: Add files via upload
Parts:
- renumbered J4 to J2, J2 to J3, J3 to J4, J9 to J6, J8 to J7, J7 to J8, J6 to J9, AC-DC_5V to Q4, + to R22, - to R23
Other:
- board text added: "+"
- board text added: "-"
Changed lines of the file:
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@@
   (general
     (thickness 1.6)
-    (drawings 10)
+    (drawings 12)
     (tracks 353)
     (zones 0)
@@
     (46 B.CrtYd user hide)
     (47 F.CrtYd user hide)
-    (48 B.Fab user)
+    (48 B.Fab user hide)
     (49 F.Fab user hide)
   )
@@
     (solder_mask_min_width 0.25)
     (aux_axis_origin 12.01 12)
-    (visible_elements 7FFFFF7F)
+    (visible_elements 7FFFFFFF)
     (pcbplotparams
       (layerselection 0x010f0_ffffffff)
@@
   (module "Library:BP pod vpaiky" (layer F.Cu)
     (at 60.744 65.694 180)
-    (fp_text reference AC-DC_5V (at 15.314 10.834 180) (layer F.SilkS)
+    (fp_text reference Q4 (at 15.314 10.834 180) (layer F.SilkS)
       (effects (font (size 1 1) (thickness 0.15)))
     )
@@
     (descr "Altech AK300 terminal block, pitch 5.0mm, 45 degree angled, see http://www.mouser.com/ds/2/16/PCBMETRC-24178.pdf")
     (tags "Altech AK300 terminal block pitch 5.0mm")
-    (fp_text reference J7 (at 2.53 -9.52) (layer F.SilkS)
+    (fp_text reference J8 (at 2.53 -9.52) (layer F.SilkS)
       (effects (font (size 1 1) (thickness 0.15)))
     )
@@
     (tags "resistor 0805")
     (attr smd)
-    (fp_text reference + (at -2.15 0) (layer B.SilkS)
+    (fp_text reference R22 (at -2.15 0) (layer B.SilkS) hide
       (effects (font (size 1 1) (thickness 0.15)) (justify mirror))
     )
@@
     (descr "Altech AK300 terminal block, pitch 5.0mm, 45 degree angled, see http://www.mouser.com/ds/2/16/PCBMETRC-24178.pdf")
     (tags "Altech AK300 terminal block pitch 5.0mm")
-    (fp_text reference J9 (at 2.55 -9.52) (layer F.SilkS)
+    (fp_text reference J6 (at 2.55 -9.52) (layer F.SilkS)
       (effects (font (size 1 1) (thickness 0.15)))
     )
@@
     (descr "Altech AK300 terminal block, pitch 5.0mm, 45 degree angled, see http://www.mouser.com/ds/2/16/PCBMETRC-24178.pdf")
     (tags "Altech AK300 terminal block pitch 5.0mm")
-    (fp_text reference J6 (at 2.55 -9.52) (layer F.SilkS)
+    (fp_text reference J9 (at 2.55 -9.52) (layer F.SilkS)
       (effects (font (size 1 1) (thickness 0.15)))
     )
@@
     (descr "Altech AK300 terminal block, pitch 5.0mm, 45 degree angled, see http://www.mouser.com/ds/2/16/PCBMETRC-24178.pdf")
     (tags "Altech AK300 terminal block pitch 5.0mm")
-    (fp_text reference J8 (at 2.57 -9.52) (layer F.SilkS)
+    (fp_text reference J7 (at 2.57 -9.52) (layer F.SilkS)
       (effects (font (size 1 1) (thickness 0.15)))
     )
@@
     (tags "resistor 0805")
     (attr smd)
-    (fp_text reference - (at -2.14 0.01) (layer B.SilkS)
+    (fp_text reference R23 (at -2.14 0.01) (layer B.SilkS) hide
       (effects (font (size 1 1) (thickness 0.15)) (justify mirror))
     )
@@
     (descr "Altech AK300 terminal block, pitch 5.0mm, 45 degree angled, see http://www.mouser.com/ds/2/16/PCBMETRC-24178.pdf")
     (tags "Altech AK300 terminal block pitch 5.0mm")
-    (fp_text reference J4 (at -3.75 5.019 180) (layer F.SilkS)
+    (fp_text reference J2 (at -3.75 5.019 180) (layer F.SilkS)
       (effects (font (size 1 1) (thickness 0.15)))
     )
@@
     (descr "Altech AK300 terminal block, pitch 5.0mm, 45 degree angled, see http://www.mouser.com/ds/2/16/PCBMETRC-24178.pdf")
     (tags "Altech AK300 terminal block pitch 5.0mm")
-    (fp_text reference J2 (at 9.192 4.106 180) (layer F.SilkS)
+    (fp_text reference J3 (at 9.192 4.106 180) (layer F.SilkS)
       (effects (font (size 1 1) (thickness 0.15)))
     )
@@
     (descr "Altech AK300 terminal block, pitch 5.0mm, 45 degree angled, see http://www.mouser.com/ds/2/16/PCBMETRC-24178.pdf")
     (tags "Altech AK300 terminal block pitch 5.0mm")
-    (fp_text reference J3 (at 2.5 9) (layer F.SilkS)
+    (fp_text reference J4 (at 2.5 9) (layer F.SilkS)
       (effects (font (size 1 1) (thickness 0.15)))
     )
@@
     )
   )
+  (gr_text + (at 64.59 103.12) (layer B.SilkS)
+    (effects (font (size 1.5 1.5) (thickness 0.3)))
+  )
+  (gr_text - (at 64.53 101.41) (layer B.SilkS)
+    (effects (font (size 1.5 1.5) (thickness 0.3)))
+  )
   (gr_line (start 12.02 105.01) (end 112.02 104.99) (layer Edge.Cuts) (width 0.12))
