File: 1.kicad_pcb (KiCad board)
At the start: 2 copper layers, 64 parts, among them J1 ValveOUT, J10 PD6, J2 MotorOUT, J3 PumpOUT, J4 220V_IN, J5 ISCP, J6 LedOUT, J7 FloatOUT, J8 SwitchOUT, J9 ButtonOUT, Q1 BT136, Q2 BT136, Q3 BT136, SW1 SW_Push, U1 ATmega8A-AU, U2 MOC3023M, U3 MOC3023M, U4 MOC3023M, Y1 16MHz

Commit message: Add files via upload
Parts:
- removed the REF** at (60.7, 65.7)
- added REF**: BP_12V, Library:MINI_PB_GERM, F.Cu at (30.9, 44.3)
- R1: footprint Resistors_SMD:R_1206 -> Resistors_SMD:R_0805
- moved D1 6.35 mm to (69.3, 51.2), turned to 180 degrees
- moved R6 6.27 mm to (65.4, 55.5)
- moved C3 6.27 mm to (63.4, 55.5)
- moved R7 4.34 mm to (81.8, 45.8)
- moved D2 4.23 mm to (81.2, 49.2)
- moved U2 4.23 mm to (85.8, 48.9)
- moved R8 3.79 mm to (76.6, 50.2)
- moved R1 0.43 mm to (40.2, 68.8)
Routing:
- net /PumpPin: track 38.6 -> 46.8 mm
- net +5V: track 132.7 -> 124.8 mm, vias 10 -> 8
- net /ValvePin: track 59.4 -> 66.9 mm
- net Net-(Q1-Pad3): track 27.4 -> 23.8 mm
- net /220_In2: track 197.2 -> 200.1 mm
- net /220_In1: track 184.8 -> 187.3 mm
- net Net-(R16-Pad2): track 4.61 -> 6.02 mm
- net /RST: track 32.2 -> 32.8 mm
- net Net-(R7-Pad1): track 3.80 -> 4.38 mm

Commit message: Add files via upload
Parts:
- removed the REF** at (30.9, 44.3)
- added AC-DC_5V: BP_12V, Library:MINI_PB_GERM, F.Cu at (30.9, 44.3)
- F1: footprint Library:MyBladeFuse -> Fuse_Holders_and_Fuses:Fuse_TE5_Littlefuse-395Series
- R2: footprint Resistors_SMD:R_1206 -> Resistors_SMD:R_0805
- moved + 9.30 mm to (62.3, 103.4), turned to 180 degrees
- moved R1 9.01 mm to (49.2, 68.2), turned to 270 degrees
- moved R3 8.47 mm to (41.9, 102.4), turned to 0 degrees
- moved R3 8.47 mm to (51.9, 102.4), turned to 0 degrees
- moved R4 8.47 mm to (31.9, 102.4), turned to 0 degrees
- moved F1 2.55 mm to (27.9, 54.2)
- renumbered R22 to +, R23 to -, R5 to R3
Routing:
- net Earth: track 316.0 -> 143.8 mm, vias 2 -> 1
- net +5V: track 124.8 -> 157.0 mm, vias 8 -> 0
- net /220_In2: track 200.1 -> 211.1 mm
- net /RST: track 32.8 -> 23.9 mm, vias 2 -> 0
- net /Switch: track 24.9 -> 28.7 mm
- net /Float: track 24.9 -> 26.5 mm
- net /PD6: track 27.9 -> 26.4 mm
- net Net-(J10-Pad1): track 7.28 -> 5.90 mm
- net Net-(F1-Pad1): track 10.4 -> 9.29 mm
- net /MOSI: track 28.3 -> 27.4 mm, vias 0 -> 1
- net /Button: track 30.1 -> 30.7 mm
- net /ValvePin: track 66.9 -> 66.8 mm, vias 2 -> 0
- added copper zone on F.Cu, net Earth
Other:
- rule via_min_size: 0.8 -> 0.1
- board text added: "+5V"
- board text added: "GND"
- board text added: "MISO"
- board text added: "MOSI"
- board text added: "RST"
- board text added: "SCK"
