File: 1.sch (KiCad schematic (older format))
At the start: 56 parts, among them J1 ValveOUT, J10 PD6, J2 MotorOUT, J3 PumpOUT, J4 220V_IN, J5 ISCP, J6 LedOUT, J7 FloatOUT, J8 SwitchOUT, J9 ButtonOUT, Q1 BT136, Q2 BT136, Q3 BT136, SW1 SW_Push, U1 ATmega8A-AU, U2 MOC3023M, U3 MOC3023M, U4 MOC3023M, Y1 16MHz

Commit message: Add files via upload
Parts:
- renumbered C9 to C7, C7 to C8, C8 to C9, D2 to D5, D4 to D6, D3 to D7, J4 to J2, J2 to J3, J3 to J4, J9 to J6, J8 to J7, J7 to J8, J6 to J9, R13 to R10, R14 to R11, R15 to R12, R16 to R13, R17 to R14, R18 to R15, R19 to R16, R20 to R17, R21 to R18, R22 to R19, R23 to R20, R12 to R21, R8 to R22, R11 to R23, R4 to R3, R3 to R4, R7 to R6, R9 to R7, R10 to R8, R6 to R9

Commit message: Add files via upload
Parts:
- removed U1: ATmega8A-AU, Housings_QFP:LQFP-32_7x7mm_Pitch0.8mm, symbol MCU_Microchip_ATmega:ATmega8A-AU
- added U1: ATmega328P-AU, Package_QFP:TQFP-32_7x7mm_P0.8mm, symbol My_ATmega:ATmega328P-AU
- C1, C2: footprint Capacitors_THT:C_Disc_D3.8mm_W2.6mm_P2.50mm -> Capacitors_SMD:C_0805
- C3, C7, C8, C9: footprint Capacitors_SMD:C_0805_HandSoldering -> Capacitors_SMD:C_0805
- D1: footprint LEDs:LED_1206_HandSoldering -> LEDs:LED_D3.0mm
- R1, R21, R22, R23, R3, R4, R5, R6, R7, R8: footprint Resistors_SMD:R_1206 -> Resistors_SMD:R_0805
- R2, R9: value 270 -> 220; footprint Resistors_SMD:R_1206 -> Resistors_SMD:R_0805
- renumbered D5 to D2, D7 to D3, D6 to D4
Connections:
- net +5V: now also U1.18 (AVCC), U1.4 (VCC), U1.6 (VCC)
- net Button: now also U1.13 (PB1)
- net Earth: now also U1.21 (GND), U1.3 (GND), U1.5 (GND)
- net Float: now also U1.11 (PD7)
- net MISO: now also U1.16 (PB4)
- net MOSI: now also U1.15 (PB3)
- net MotorPin: now also U1.9 (PD5)
- net PD6: now also U1.10 (PD6)
- net PumpPin: now also U1.32 (PD2)
- net RST: now also U1.29 (~RESET~/PC6)
- net SCK: now also U1.17 (PB5)
- net Switch: now also U1.12 (PB0)
- net ValvePin: now also U1.31 (PD1)
- net at C1.1, Y1.1: now also U1.8 (XTAL2/PB7)
- net at C2.1, Y1.2: now also U1.7 (XTAL1/PB6)
- net at R2.2: now also U1.14 (PB2)
Other:
- moved on the sheet: C1, C2, C3, R1, R2, R3, R4, R5, SW1, Y1

Commit message: Add files via upload
Parts:
- added Q4: power_block-My_library, Library:BP pod vpaiky, symbol My_library:AC-DC
- renumbered C8 to C7, C9 to C8, C7 to C9, R8 to R10, R23 to R11, R21 to R12, R10 to R13, R11 to R14, R12 to R15, R13 to R16, R14 to R17, R15 to R18, R16 to R19, R17 to R20, R18 to R21, R19 to R22, R20 to R23, R4 to R3, R3 to R4, R9 to R6, R6 to R7, R22 to R8, R7 to R9
Connections:
- net +5V: now also Q4.3 (OUT+)
- net 220_In1: now also Q4.1 (IN_1)
- net 220_In2: now also Q4.2 (IN_2)
- net Earth: now also Q4.4 (OUT-)
Changed lines of the file:
@@
 	2205 2095 2475 2095
-Wire Wire Line
-	2475 2095 2475 2123
 Wire Wire Line
 	2475 2325 2475 2395
@@
 Wire Wire Line
 	2255 1735 2475 1735
-Wire Wire Line
-	2475 1735 2475 1923
 Connection ~ 2475 1735
 $Comp
@@
 $EndComp
 $Comp
-L Device:C C8
+L Device:C C7
 U 1 1 5DF97454
 P 8295 2780
-F 0 "C8" H 8350 2685 50  0000 C CNN
+F 0 "C7" H 8350 2685 50  0000 C CNN
 F 1 "0.33uF" V 8165 2775 50  0000 C CNN
 F 2 "Capacitors_SMD:C_0805" H 8333 2630 50  0001 C CNN
@@
 $EndComp
 $Comp
-L Device:C C9
+L Device:C C8
 U 1 1 5DF9EE90
 P 8295 3265
-F 0 "C9" H 8350 3170 50  0000 C CNN
+F 0 "C8" H 8350 3170 50  0000 C CNN
 F 1 "0.33uF" V 8165 3260 50  0000 C CNN
 F 2 "Capacitors_SMD:C_0805" H 8333 3115 50  0001 C CNN
@@
 $EndComp
 $Comp
-L Device:C C7
+L Device:C C9
 U 1 1 5DFAB79A
 P 8305 2320
-F 0 "C7" H 8360 2225 50  0000 C CNN
+F 0 "C9" H 8360 2225 50  0000 C CNN
 F 1 "0.33uF" V 8175 2315 50  0000 C CNN
 F 2 "Capacitors_SMD:C_0805" H 8343 2170 50  0001 C CNN
@@
 $EndComp
 $Comp
-L Device:R R9
+L Device:R R6
 U 1 1 5DFE1740
 P 4895 4895
-F 0 "R9" V 4820 4895 50  0000 C CNN
+F 0 "R6" V 4820 4895 50  0000 C CNN
 F 1 "220" V 4895 4895 50  0000 C CNN
 F 2 "Resistors_SMD:R_0805" V 4825 4895 50  0001 C CNN
@@
 $EndComp
 $Comp
-L Device:R R8
+L Device:R R10
 U 1 1 5DEE37F8
 P 5380 3240
-F 0 "R8" V 5305 3240 50  0000 C CNN
+F 0 "R10" V 5305 3240 50  0000 C CNN
 F 1 "220" V 5380 3240 50  0000 C CNN
 F 2 "Resistors_SMD:R_0805" V 5310 3240 50  0001 C CNN
@@
 $EndComp
 $Comp
-L Device:R R15
+L Device:R R18
 U 1 1 5DEE37EB
 P 6670 3240
-F 0 "R15" V 6590 3240 50  0000 C CNN
+F 0 "R18" V 6590 3240 50  0000 C CNN
 F 1 "390" V 6670 3240 50  0000 C CNN
 F 2 "Resistors_THT:R_Axial_DIN0414_L11.9mm_D4.5mm_P15.24mm_Horizontal" V 6600 3240 50  0001 C CNN
@@
 	6520 3240 6470 3240
 $Comp
-L Device:R R12
+L Device:R R15
 U 1 1 5DEE37DE
 P 6470 3680
-F 0 "R12" H 6355 3685 50  0000 C CNN
+F 0 "R15" H 6355 3685 50  0000 C CNN
 F 1 "330" V 6465 3680 50  0000 C CNN
 F 2 "Resistors_THT:R_Axial_DIN0414_L11.9mm_D4.5mm_P15.24mm_Horizontal" V 6400 3680 50  0001 C CNN
@@
 $EndComp
 $Comp
-L Device:R R18
+L Device:R R21
 U 1 1 5DEE37D8
 P 7200 3390
-F 0 "R18" H 7085 3400 50  0000 C CNN
+F 0 "R21" H 7085 3400 50  0000 C CNN
 F 1 "39" V 7195 3390 50  0000 C CNN
 F 2 "Resistors_THT:R_Axial_DIN0414_L11.9mm_D4.5mm_P15.24mm_Horizontal" V 7130 3390 50  0001 C CNN
@@
 $EndComp
 $Comp
-L Device:R R13
+L Device:R R16
 U 1 1 5DECB46F
 P 6670 1620
-F 0 "R13" V 6590 1620 50  0000 C CNN
+F 0 "R16" V 6590 1620 50  0000 C CNN
 F 1 "390" V 6670 1620 50  0000 C CNN
 F 2 "Resistors_THT:R_Axial_DIN0414_L11.9mm_D4.5mm_P15.24mm_Horizontal" V 6600 1620 50  0001 C CNN
@@
 	6520 1620 6470 1620
 $Comp
-L Device:R R10
+L Device:R R13
 U 1 1 5DECB47C
 P 6470 2060
-F 0 "R10" H 6355 2060 50  0000 C CNN
+F 0 "R13" H 6355 2060 50  0000 C CNN
 F 1 "330" V 6465 2060 50  0000 C CNN
 F 2 "Resistors_THT:R_Axial_DIN0414_L11.9mm_D4.5mm_P15.24mm_Horizontal" V 6400 2060 50  0001 C CNN
@@
 $EndComp
 $Comp
-L Device:R R16
+L Device:R R19
 U 1 1 5DECB482
 P 7200 1770
-F 0 "R16" H 7085 1770 50  0000 C CNN
+F 0 "R19" H 7085 1770 50  0000 C CNN
 F 1 "39" V 7195 1770 50  0000 C CNN
 F 2 "Resistors_THT:R_Axial_DIN0414_L11.9mm_D4.5mm_P15.24mm_Horizontal" V 7130 1770 50  0001 C CNN
@@
 Pump
 $Comp
-L Device:R R6
+L Device:R R7
 U 1 1 5DECB461
 P 5380 1620
-F 0 "R6" V 5305 1620 50  0000 C CNN
+F 0 "R7" V 5305 1620 50  0000 C CNN
 F 1 "220" V 5380 1620 50  0000 C CNN
 F 2 "Resistors_SMD:R_0805" V 5310 1620 50  0001 C CNN
@@
 $EndComp
 $Comp
-L Device:R R7
+L Device:R R9
 U 1 1 5DE86323
 P 5380 2430
-F 0 "R7" V 5305 2430 50  0000 C CNN
+F 0 "R9" V 5305 2430 50  0000 C CNN
 F 1 "220" V 5380 2430 50  0000 C CNN
 F 2 "Resistors_SMD:R_0805" V 5310 2430 50  0001 C CNN
@@
 	0    1    1    0
 $EndComp
+Wire Wire Line
+	6520 2430 6470 2430
 $Comp
 L Device:R R14
-U 1 1 5DE8A46C
-P 6670 2430
-F 0 "R14" V 6590 2430 50  0000 C CNN
-F 1 "390" V 6670 2430 50  0000 C CNN
-F 2 "Resistors_THT:R_Axial_DIN0414_L11.9mm_D4.5mm_P15.24mm_Horizontal" V 6600 2430 50  0001 C CNN
-F 3 "~" H 6670 2430 50  0001 C CNN
-	1    6670 2430
-	0    1    1    0
-$EndComp
-Wire Wire Line
-	6520 2430 6470 2430
-$Comp
-L Device:R R11
 U 1 1 5DE90BC5
 P 6470 2870
-F 0 "R11" H 6355 2880 50  0000 C CNN
+F 0 "R14" H 6355 2880 50  0000 C CNN
 F 1 "330" V 6465 2870 50  0000 C CNN
 F 2 "Resistors_THT:R_Axial_DIN0414_L11.9mm_D4.5mm_P15.24mm_Horizontal" V 6400 2870 50  0001 C CNN
@@
 $EndComp
 $Comp
-L Device:R R17
+L Device:R R20
 U 1 1 5DE9194E
 P 7200 2580
-F 0 "R17" H 7075 2590 50  0000 C CNN
+F 0 "R20" H 7075 2590 50  0000 C CNN
 F 1 "39" V 7195 2580 50  0000 C CNN
 F 2 "Resistors_THT:R_Axial_DIN0414_L11.9mm_D4.5mm_P15.24mm_Horizontal" V 7130 2580 50  0001 C CNN
@@
 PD6
 $Comp
-L Device:R_Small R20
+L Device:R_Small R23
 U 1 1 5DED3415
 P 8485 4045
-F 0 "R20" V 8485 4045 50  0000 C CNN
+F 0 "R23" V 8485 4045 50  0000 C CNN
 F 1 "R" V 8535 4140 50  0000 C CNN
 F 2 "Resistors_SMD:R_0805" H 8485 4045 50  0001 C CNN
@@
 Connection ~ 5870 3440
 $Comp
-L Device:R_Small R19
+L Device:R_Small R22
 U 1 1 5DEE6BEA
 P 8485 3965
-F 0 "R19" V 8485 3965 50  0000 C CNN
+F 0 "R22" V 8485 3965 50  0000 C CNN
 F 1 "R" V 8450 4060 50  0000 C CNN
 F 2 "Resistors_SMD:R_0805" H 8485 3965 50  0001 C CNN
@@
 $EndComp
 $Comp
-L My_library:AC-DC #Q4
+L My_library:AC-DC Q4
 U 1 1 5DEDCE5A
 P 5495 5195
-F 0 "#Q4" H 5490 4785 50  0000 C CNN
+F 0 "Q4" H 5490 4785 50  0000 C CNN
 F 1 "power_block-My_library" H 5495 4985 50  0000 C CNN
 F 2 "Library:BP pod vpaiky" H 5495 5195 50  0001 C CNN
@@
 Connection ~ 5870 2630
 $Comp
-L Device:R R21
+L Device:R R12
 U 1 1 5DEB00E1
 P 5420 2630
-F 0 "R21" V 5345 2630 50  0000 C CNN
+F 0 "R12" V 5345 2630 50  0000 C CNN
 F 1 "220" V 5420 2630 50  0000 C CNN
 F 2 "Resistors_SMD:R_0805" V 5350 2630 50  0001 C CNN
@@
 	5230 2630 5230 2430
 $Comp
-L Device:R R22
+L Device:R R8
 U 1 1 5DEEB711
 P 5380 1820
-F 0 "R22" V 5305 1820 50  0000 C CNN
+F 0 "R8" V 5305 1820 50  0000 C CNN
 F 1 "220" V 5380 1820 50  0000 C CNN
 F 2 "Resistors_SMD:R_0805" V 5310 1820 50  0001 C CNN
@@
 $EndComp
 $Comp
-L Device:R R23
+L Device:R R11
 U 1 1 5DEF08D2
 P 5380 3440
-F 0 "R23" V 5305 3440 50  0000 C CNN
+F 0 "R11" V 5305 3440 50  0000 C CNN
 F 1 "220" V 5380 3440 50  0000 C CNN
 F 2 "Resistors_SMD:R_0805" V 5310 3440 50  0001 C CNN
@@
 	4020 1860 3765 1860
 $Comp
-L Device:R R4
+L Device:R R3
 U 1 1 5DF5A9F9
 P 4170 1860
-F 0 "R4" V 4090 1860 50  0000 C CNN
+F 0 "R3" V 4090 1860 50  0000 C CNN
 F 1 "150k" V 4170 1860 50  0000 C CNN
 F 2 "Resistors_SMD:R_0805" V 4100 1860 50  0001 C CNN
@@
 Connection ~ 4320 1860
 Wire Wire Line
-	3675 1925 3675 1923
-Wire Wire Line
 	3765 1960 4000 1960
 Wire Wire Line
 	3765 1990 3765 1960
 $Comp
-L Device:R R3
+L Device:R R4
 U 1 1 5DE7B4F3
 P 4170 1990
-F 0 "R3" V 4210 2155 50  0000 C CNN
+F 0 "R4" V 4210 2155 50  0000 C CNN
 F 1 "150k" V 4170 1990 50  0000 C CNN
 F 2 "Resistors_SMD:R_0805" V 4100 1990 50  0001 C CNN
@@
 Wire Wire Line
 	4020 1990 3765 1990
-Wire Wire Line
-	3675 1990 3675 2023
 Connection ~ 3765 1990
 Wire Wire Line
 	3765 1990 3675 1990
-Wire Wire Line
-	3675 2105 3675 2123
 Connection ~ 5230 3240
 Wire Wire Line
@@
 	1    0    0    -1
 $EndComp
-Wire Wire Line
-	3075 1625 3174 1625
-Connection ~ 3675 1923
-Wire Wire Line
-	3675 1923 3675 1860
-Connection ~ 3675 2023
-Wire Wire Line
-	3675 2023 3675 2025
-Connection ~ 3675 2123
-Wire Wire Line
-	3675 2123 3675 2125
-Connection ~ 2475 1923
-Wire Wire Line
-	2475 1923 2475 1925
-Connection ~ 2475 2123
-Wire Wire Line
-	2475 2123 2475 2125
-Connection ~ 3174 1625
-Wire Wire Line
-	3174 1625 3175 1625
 Connection ~ 3075 4425
 Connection ~ 3075 1625
+Wire Wire Line
+	2475 2095 2475 2125
+Wire Wire Line
+	2475 1735 2475 1925
+Wire Wire Line
+	3675 1860 3675 1925
+Wire Wire Line
+	3675 1990 3675 2025
+Wire Wire Line
+	3675 2105 3675 2125
+Wire Wire Line
+	3075 1625 3175 1625
+$Comp
+L Device:R R17
+U 1 1 5DE8A46C
+P 6670 2430
+F 0 "R17" V 6590 2430 50  0000 C CNN
+F 1 "390" V 6670 2430 50  0000 C CNN
+F 2 "Resistors_THT:R_Axial_DIN0414_L11.9mm_D4.5mm_P15.24mm_Horizontal" V 6600 2430 50  0001 C CNN
+F 3 "~" H 6670 2430 50  0001 C CNN
+	1    6670 2430
+	0    1    1    0
+$EndComp
 $EndSCHEMATC
