File: 1.sch (KiCad schematic (older format))
At the start: 56 parts, among them J1 ValveOUT, J10 PD6, J2 MotorOUT, J3 PumpOUT, J4 220V_IN, J5 ISCP, J6 LedOUT, J7 FloatOUT, J8 SwitchOUT, J9 ButtonOUT, Q1 BT136, Q2 BT136, Q3 BT136, SW1 SW_Push, U1 ATmega8A-AU, U2 MOC3023M, U3 MOC3023M, U4 MOC3023M, Y1 16MHz

Commit message: Add files via upload
Changed lines of the file:
@@
 	1770 2290 1770 2590
-$Comp
-L power:Earth #PWR01
-U 1 1 5DE643F3
-P 1680 2590
-F 0 "#PWR01" H 1680 2340 50  0001 C CNN
-F 1 "Earth" H 1680 2440 50  0001 C CNN
-F 2 "" H 1680 2590 50  0001 C CNN
-F 3 "~" H 1680 2590 50  0001 C CNN
-	1    1680 2590
-	1    0    0    -1
-$EndComp
 $Comp
 L power:+5V #PWR06
@@
 	1    0    0    -1
 $EndComp
-$Comp
-L power:Earth #PWR07
-U 1 1 5DE65D52
-P 3095 4620
-F 0 "#PWR07" H 3095 4370 50  0001 C CNN
-F 1 "Earth" H 3095 4470 50  0001 C CNN
-F 2 "" H 3095 4620 50  0001 C CNN
-F 3 "~" H 3095 4620 50  0001 C CNN
-	1    3095 4620
-	1    0    0    -1
-$EndComp
 Wire Wire Line
 	3195 4620 3095 4620
@@
 $EndComp
 $Comp
-L power:Earth #PWR04
-U 1 1 5DE68298
-P 2140 3670
-F 0 "#PWR04" H 2140 3420 50  0001 C CNN
-F 1 "Earth" H 2140 3520 50  0001 C CNN
-F 2 "" H 2140 3670 50  0001 C CNN
-F 3 "~" H 2140 3670 50  0001 C CNN
-	1    2140 3670
-	1    0    0    -1
-$EndComp
-$Comp
 L Device:C C3
 U 1 1 5DE6885E
@@
 	2495 1930 2495 2120
 Connection ~ 2495 1930
-$Comp
-L power:Earth #PWR02
-U 1 1 5DE75AD2
-P 1875 1930
-F 0 "#PWR02" H 1875 1680 50  0001 C CNN
-F 1 "Earth" H 1875 1780 50  0001 C CNN
-F 2 "" H 1875 1930 50  0001 C CNN
-F 3 "~" H 1875 1930 50  0001 C CNN
-	1    1875 1930
-	1    0    0    -1
-$EndComp
 Wire Wire Line
 	2495 2120 2350 2120
@@
 	1    0    0    -1
 $EndComp
-$Comp
-L power:Earth #PWR022
-U 1 1 5DE82930
-P 8925 1985
-F 0 "#PWR022" H 8925 1735 50  0001 C CNN
-F 1 "Earth" H 8925 1835 50  0001 C CNN
-F 2 "" H 8925 1985 50  0001 C CNN
-F 3 "~" H 8925 1985 50  0001 C CNN
-	1    8925 1985
-	1    0    0    -1
-$EndComp
 Wire Wire Line
 	3695 2420 3870 2420
@@
 $EndComp
 Connection ~ 2495 2120
-Connection ~ 3095 4620
 Connection ~ 3095 1820
 $Comp
@@
 Wire Wire Line
 	3695 3720 4020 3720
+$Comp
+L power:GNDA #PWR0101
+U 1 1 5E1E0969
+P 3095 4620
+F 0 "#PWR0101" H 3095 4370 50  0001 C CNN
+F 1 "GNDA" H 3100 4447 50  0000 C CNN
+F 2 "" H 3095 4620 50  0001 C CNN
+F 3 "" H 3095 4620 50  0001 C CNN
+	1    3095 4620
+	1    0    0    -1
+$EndComp
+Connection ~ 3095 4620
+$Comp
+L power:GNDA #PWR0102
+U 1 1 5E1F4FB2
+P 5115 4530
+F 0 "#PWR0102" H 5115 4280 50  0001 C CNN
+F 1 "GNDA" H 5120 4357 50  0000 C CNN
+F 2 "" H 5115 4530 50  0001 C CNN
+F 3 "" H 5115 4530 50  0001 C CNN
+	1    5115 4530
+	1    0    0    -1
+$EndComp
+Wire Wire Line
+	5115 4530 5045 4530
+Connection ~ 5045 4530
+$Comp
+L power:GNDA #PWR0103
+U 1 1 5E1FAE32
+P 2140 3670
+F 0 "#PWR0103" H 2140 3420 50  0001 C CNN
+F 1 "GNDA" H 2145 3497 50  0000 C CNN
+F 2 "" H 2140 3670 50  0001 C CNN
+F 3 "" H 2140 3670 50  0001 C CNN
+	1    2140 3670
+	1    0    0    -1
+$EndComp
+$Comp
+L power:GNDA #PWR0104
+U 1 1 5E1FB4B1
+P 1875 1930
+F 0 "#PWR0104" H 1875 1680 50  0001 C CNN
+F 1 "GNDA" H 1720 1930 50  0000 C CNN
+F 2 "" H 1875 1930 50  0001 C CNN
+F 3 "" H 1875 1930 50  0001 C CNN
+	1    1875 1930
+	1    0    0    -1
+$EndComp
+$Comp
+L power:GNDA #PWR0105
+U 1 1 5E200B7F
+P 1680 2590
+F 0 "#PWR0105" H 1680 2340 50  0001 C CNN
+F 1 "GNDA" H 1525 2590 50  0000 C CNN
+F 2 "" H 1680 2590 50  0001 C CNN
+F 3 "" H 1680 2590 50  0001 C CNN
+	1    1680 2590
+	1    0    0    -1
+$EndComp
+$Comp
+L power:GNDA #PWR0106
+U 1 1 5E200EBD
+P 8925 1985
+F 0 "#PWR0106" H 8925 1735 50  0001 C CNN
+F 1 "GNDA" H 9065 2035 50  0000 C CNN
+F 2 "" H 8925 1985 50  0001 C CNN
+F 3 "" H 8925 1985 50  0001 C CNN
+	1    8925 1985
+	1    0    0    -1
+$EndComp
 $EndSCHEMATC
